File: smart-bell-pcb-esp32.kicad_pcb (KiCad board)
At the start: 2 copper layers, 0 parts

Commit message: feat: update sketch
Parts:
- added C1: C_Polarized_US, Capacitor_THT:CP_Radial_D8.0mm_P3.50mm, F.Cu at (121.0, 138.0)
- added D1: 1N4007, Diode_THT:D_DO-41_SOD81_P10.16mm_Horizontal, F.Cu at (121.3, 104.0)
- added J1: Barrel_Jack_MountingPin, Connector_BarrelJack:BarrelJack_Horizontal, F.Cu at (110.6, 138.6)
- added J2: Screw_Terminal_01x03, TerminalBlock_Phoenix:TerminalBlock_Phoenix_PT-1,5-3-5.0-H_1x03_P5.00mm_Horizontal, F.Cu at (99.6, 127.2)
- added J3: Conn_01x04, Connector_PinHeader_2.54mm:PinHeader_1x05_P2.54mm_Vertical, F.Cu at (115.5, 135.6)
- added K1: FINDER-40.11, Relay_THT:Relay_SPDT_Finder_40.11, F.Cu at (102.9, 67.7)
- added Q1: BC547, Package_TO_SOT_THT:TO-92_Inline, F.Cu at (102.0, 109.5)
- added R1: R, Resistor_THT:R_Axial_DIN0207_L6.3mm_D2.5mm_P10.16mm_Horizontal, F.Cu at (114.7, 124.2)
- added R2: R, Resistor_THT:R_Axial_DIN0207_L6.3mm_D2.5mm_P10.16mm_Horizontal, F.Cu at (114.7, 128.2)
- added U1: ESP32_DEVKIT_V1, customLibraries:ESP32_DEVKIT_V1, F.Cu at (84.0, 89.9)

Commit message: s
Parts:
- moved J3 30.9 mm to (90.5, 117.4)
- moved C1 28.3 mm to (99.2, 120.0), turned to 180 degrees
- moved Q1 19.9 mm to (96.0, 128.5)
- moved R1 19.6 mm to (106.5, 106.5)
- moved R2 19.6 mm to (106.5, 110.5)
- moved J2 19.6 mm to (91.4, 109.5)
- moved U1 18.8 mm to (71.8, 104.2), turned to 180 degrees
- moved K1 16.8 mm to (92.0, 80.5)
- moved D1 13.8 mm to (116.6, 117.0), turned to 180 degrees
- moved J1 13.4 mm to (116.5, 126.5)
Routing:
- net +5V: track 0.00 -> 9.53 mm
