File: smart-bell-pcb-esp32.kicad_sch (KiCad schematic)
At the start: 10 parts, among them J1 Barrel_Jack_MountingPin, J2 Screw_Terminal_01x03, J3 Conn_01x04, K1 FINDER-40.11, Q1 BC547, U1 ESP32_DEVKIT_V1

Commit message: s
Other:
- moved on the sheet: C1, J1, J3, U1
